File: PCD_Design/LCD/lcd.brd (EAGLE design)
At the start: 155.9 x 114.3 mm, 7 parts

Commit message: manglet en kobling
Connections:
- removed net N$5: PH1.2, R1.P$2
- net N$4: now also PH1.2, R1.P$2
Routing:
- net N$4: track 141.6 -> 169.7 mm
- net N$5: track 15.4 -> 0.00 mm
Changed lines of the file:
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@@
 <wire x1="99.695" y1="49.53" x2="99.695" y2="36.205" width="0.1524" layer="16"/>
 <wire x1="92.45" y1="28.96" x2="99.695" y2="36.205" width="0.1524" layer="16"/>
-</signal>
-<signal name="N$5">
 <contactref element="PH1" pad="2"/>
 <contactref element="R1" pad="P$2"/>
@@
 <wire x1="54.61" y1="86.36" x2="39.37" y2="86.36" width="0.1524" layer="1"/>
 <wire x1="39.37" y1="86.36" x2="39.29" y2="86.32" width="0.1524" layer="1"/>
+<wire x1="67.295" y1="86.36" x2="54.61" y2="86.36" width="0.1524" layer="16"/>
 </signal>
 <signal name="N$6">
